File: PCB/WaterCirculation/WaterCirculation.sch (EAGLE design)
At the start: 27 parts, among them K1 G5V1, K2 G5V1, K3 G5V1, Q2 MPSA42, Q3 MPSA42

Commit message: Board Layout
Not finialized
Parts:
- removed D3: (no value), diode:DIODE-SOD123
- removed LED3: (no value), led:LEDCHIP-LED0805
- added D1: (no value), diode:DIODE-SOD123
- added LED1: (no value), led:LEDCHIP-LED0805
- renumbered Q2 to Q1
Connections:
- net +5V: now also D1.C; no longer D3.C
- net N$2: now also D1.A, LED1.C; no longer D2.A, LED2.C
- net N$3: now also LED1.A; no longer LED2.A
- net N$7: now also D2.A, LED2.C; no longer D3.A, LED3.C
- net N$8: now also LED2.A; no longer LED3.A
Other:
- moved on the sheet: D2, LED2
Changed lines of the file:
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@@
 <part name="U$1" library="diy-modules" deviceset="WEMOS-D1-MINI" device=""/>
 <part name="K1" library="relay" deviceset="G5V1" device=""/>
-<part name="D2" library="diode" deviceset="DIODE-" device="SOD123"/>
+<part name="D1" library="diode" deviceset="DIODE-" device="SOD123"/>
 <part name="R6" library="resistor" deviceset="R-US_" device="R0805" value="1k"/>
-<part name="LED2" library="led" deviceset="LED" device="CHIP-LED0805"/>
+<part name="LED1" library="led" deviceset="LED" device="CHIP-LED0805"/>
 <part name="P+1" library="supply1" deviceset="+5V" device=""/>
-<part name="Q2" library="SparkFun-DiscreteSemi" deviceset="TRANSISTOR_NPN" device="MPSA42" value="MPSA42"/>
+<part name="Q1" library="SparkFun-DiscreteSemi" deviceset="TRANSISTOR_NPN" device="MPSA42" value="MPSA42"/>
 <part name="GND1" library="supply1" deviceset="GND" device=""/>
 <part name="R4" library="resistor" deviceset="R-US_" device="R0805" value="1k"/>
 <part name="K3" library="relay" deviceset="G5V1" device=""/>
-<part name="D3" library="diode" deviceset="DIODE-" device="SOD123"/>
+<part name="D2" library="diode" deviceset="DIODE-" device="SOD123"/>
 <part name="R3" library="resistor" deviceset="R-US_" device="R0805" value="1k"/>
-<part name="LED3" library="led" deviceset="LED" device="CHIP-LED0805"/>
+<part name="LED2" library="led" deviceset="LED" device="CHIP-LED0805"/>
 <part name="P+3" library="supply1" deviceset="+5V" device=""/>
 <part name="Q3" library="SparkFun-DiscreteSemi" deviceset="TRANSISTOR_NPN" device="MPSA42" value="MPSA42"/>
@@
 <attribute name="PART" x="116.84" y="96.52" size="1.778" layer="95"/>
 </instance>
-<instance part="D2" gate="G$1" x="101.6" y="60.96" smashed="yes" rot="R90">
+<instance part="D1" gate="G$1" x="101.6" y="60.96" smashed="yes" rot="R90">
 <attribute name="NAME" x="101.1174" y="63.5" size="1.778" layer="95" rot="R90"/>
 <attribute name="VALUE" x="103.9114" y="63.5" size="1.778" layer="96" rot="R90"/>
@@
 <attribute name="VALUE" x="97.282" y="62.23" size="1.778" layer="96" rot="R90"/>
 </instance>
-<instance part="LED2" gate="G$1" x="93.98" y="55.88" smashed="yes">
+<instance part="LED1" gate="G$1" x="93.98" y="55.88" smashed="yes">
 <attribute name="NAME" x="97.536" y="51.308" size="1.778" layer="95" rot="R90"/>
 <attribute name="VALUE" x="99.695" y="51.308" size="1.778" layer="96" rot="R90"/>
@@
 <attribute name="VALUE" x="96.52" y="78.74" size="1.778" layer="96" rot="R90"/>
 </instance>
-<instance part="Q2" gate="G$1" x="96.52" y="40.64" smashed="yes">
+<instance part="Q1" gate="G$1" x="96.52" y="40.64" smashed="yes">
 <attribute name="NAME" x="101.6" y="40.64" size="1.778" layer="95"/>
 <attribute name="VALUE" x="101.6" y="38.1" size="1.778" layer="96"/>
@@
 <attribute name="PART" x="162.56" y="99.06" size="1.778" layer="95"/>
 </instance>
-<instance part="D3" gate="G$1" x="160.02" y="60.96" smashed="yes" rot="R90">
+<instance part="D2" gate="G$1" x="160.02" y="60.96" smashed="yes" rot="R90">
 <attribute name="NAME" x="159.5374" y="63.5" size="1.778" layer="95" rot="R90"/>
 <attribute name="VALUE" x="162.3314" y="63.5" size="1.778" layer="96" rot="R90"/>
@@
 <attribute name="VALUE" x="155.702" y="62.23" size="1.778" layer="96" rot="R90"/>
 </instance>
-<instance part="LED3" gate="G$1" x="152.4" y="55.88" smashed="yes">
+<instance part="LED2" gate="G$1" x="152.4" y="55.88" smashed="yes">
 <attribute name="NAME" x="155.956" y="51.308" size="1.778" layer="95" rot="R90"/>
 <attribute name="VALUE" x="158.115" y="51.308" size="1.778" layer="96" rot="R90"/>
@@
 <net name="N$2" class="0">
 <segment>
-<pinref part="D2" gate="G$1" pin="A"/>
+<pinref part="D1" gate="G$1" pin="A"/>
 <wire x1="101.6" y1="58.42" x2="101.6" y2="53.34" width="0.1524" layer="91"/>
 <pinref part="K1" gate="1" pin="2"/>
 <wire x1="101.6" y1="53.34" x2="109.22" y2="53.34" width="0.1524" layer="91"/>
 <wire x1="109.22" y1="53.34" x2="109.22" y2="55.88" width="0.1524" layer="91"/>
-<pinref part="LED2" gate="G$1" pin="C"/>
+<pinref part="LED1" gate="G$1" pin="C"/>
 <wire x1="93.98" y1="50.8" x2="93.98" y2="48.26" width="0.1524" layer="91"/>
 <wire x1="93.98" y1="48.26" x2="99.06" y2="48.26" width="0.1524" layer="91"/>
@@
 <wire x1="101.6" y1="48.26" x2="101.6" y2="53.34" width="0.1524" layer="91"/>
 <junction x="101.6" y="53.34"/>
-<pinref part="Q2" gate="G$1" pin="C"/>
+<pinref part="Q1" gate="G$1" pin="C"/>
 <wire x1="99.06" y1="45.72" x2="99.06" y2="48.26" width="0.1524" layer="91"/>
 <junction x="99.06" y="48.26"/>
@@
 <wire x1="93.98" y1="76.2" x2="93.98" y2="71.12" width="0.1524" layer="91"/>
 <wire x1="93.98" y1="76.2" x2="99.06" y2="76.2" width="0.1524" layer="91"/>
-<pinref part="D2" gate="G$1" pin="C"/>
+<pinref part="D1" gate="G$1" pin="C"/>
 <wire x1="99.06" y1="76.2" x2="101.6" y2="76.2" width="0.1524" layer="91"/>
 <wire x1="101.6" y1="63.5" x2="101.6" y2="68.58" width="0.1524" layer="91"/>
@@
 <wire x1="152.4" y1="76.2" x2="152.4" y2="71.12" width="0.1524" layer="91"/>
 <wire x1="152.4" y1="76.2" x2="157.48" y2="76.2" width="0.1524" layer="91"/>
-<pinref part="D3" gate="G$1" pin="C"/>
+<pinref part="D2" gate="G$1" pin="C"/>
 <wire x1="157.48" y1="76.2" x2="160.02" y2="76.2" width="0.1524" layer="91"/>
 <wire x1="160.02" y1="63.5" x2="160.02" y2="68.58" width="0.1524" layer="91"/>
@@
 <segment>
 <pinref part="R6" gate="G$1" pin="1"/>
-<pinref part="LED2" gate="G$1" pin="A"/>
+<pinref part="LED1" gate="G$1" pin="A"/>
 <wire x1="93.98" y1="60.96" x2="93.98" y2="58.42" width="0.1524" layer="91"/>
 </segment>
@@
 <net name="GND" class="0">
 <segment>
-<pinref part="Q2" gate="G$1" pin="E"/>
+<pinref part="Q1" gate="G$1" pin="E"/>
 <pinref part="GND1" gate="1" pin="GND"/>
 <wire x1="99.06" y1="35.56" x2="99.06" y2="33.02" width="0.1524" layer="91"/>
@@
 <segment>
 <pinref part="R4" gate="G$1" pin="1"/>
-<pinref part="Q2" gate="G$1" pin="B"/>
+<pinref part="Q1" gate="G$1" pin="B"/>
 <wire x1="91.44" y1="40.64" x2="93.98" y2="40.64" width="0.1524" layer="91"/>
 </segment>
@@
 <net name="N$7" class="0">
 <segment>
-<pinref part="D3" gate="G$1" pin="A"/>
+<pinref part="D2" gate="G$1" pin="A"/>
 <wire x1="160.02" y1="58.42" x2="160.02" y2="53.34" width="0.1524" layer="91"/>
 <pinref part="K3" gate="1" pin="2"/>
 <wire x1="160.02" y1="53.34" x2="167.64" y2="53.34" width="0.1524" layer="91"/>
 <wire x1="167.64" y1="53.34" x2="167.64" y2="55.88" width="0.1524" layer="91"/>
-<pinref part="LED3" gate="G$1" pin="C"/>
+<pinref part="LED2" gate="G$1" pin="C"/>
 <wire x1="152.4" y1="50.8" x2="152.4" y2="48.26" width="0.1524" layer="91"/>
 <wire x1="152.4" y1="48.26" x2="157.48" y2="48.26" width="0.1524" layer="91"/>
@@
 <segment>
 <pinref part="R3" gate="G$1" pin="1"/>
-<pinref part="LED3" gate="G$1" pin="A"/>
+<pinref part="LED2" gate="G$1" pin="A"/>
 <wire x1="152.4" y1="60.96" x2="152.4" y2="58.42" width="0.1524" layer="91"/>
 </segment>

Commit message: final layout
Parts:
- added 110INB: (no value), SparkFun-Connectors:M023.5MM
Connections:
- net N$10: now also 110INB.1
- net N$6: now also 110INB.2
Changed lines of the file:
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@@
 <part name="STATUSLED" library="SparkFun-Connectors" deviceset="M02" device="3.5MM"/>
 <part name="R2" library="resistor" deviceset="R-US_" device="R0805" value="1k"/>
+<part name="110INB" library="SparkFun-Connectors" deviceset="M02" device="3.5MM"/>
 </parts>
 <sheets>
@@
 <attribute name="NAME" x="-34.29" y="62.0014" size="1.778" layer="95" rot="R180"/>
 <attribute name="VALUE" x="-34.29" y="66.802" size="1.778" layer="96" rot="R180"/>
+</instance>
+<instance part="110INB" gate="G$1" x="134.62" y="124.46" smashed="yes" rot="R270">
+<attribute name="VALUE" x="129.54" y="127" size="1.778" layer="96" rot="R270"/>
+<attribute name="NAME" x="140.462" y="127" size="1.778" layer="95" rot="R270"/>
 </instance>
 </instances>
@@
 <segment>
 <pinref part="110IN" gate="G$1" pin="2"/>
-<wire x1="149.86" y1="116.84" x2="149.86" y2="111.76" width="0.1524" layer="91"/>
+<wire x1="149.86" y1="116.84" x2="149.86" y2="114.3" width="0.1524" layer="91"/>
+<wire x1="149.86" y1="114.3" x2="149.86" y2="111.76" width="0.1524" layer="91"/>
 <wire x1="149.86" y1="111.76" x2="172.72" y2="111.76" width="0.1524" layer="91"/>
 <pinref part="PUMPOUT" gate="G$1" pin="2"/>
 <wire x1="172.72" y1="111.76" x2="172.72" y2="116.84" width="0.1524" layer="91"/>
+<pinref part="110INB" gate="G$1" pin="2"/>
+<wire x1="137.16" y1="116.84" x2="137.16" y2="114.3" width="0.1524" layer="91"/>
+<wire x1="137.16" y1="114.3" x2="149.86" y2="114.3" width="0.1524" layer="91"/>
+<junction x="149.86" y="114.3"/>
 </segment>
 </net>
@@
 <wire x1="147.32" y1="116.84" x2="147.32" y2="104.14" width="0.1524" layer="91"/>
 <wire x1="147.32" y1="104.14" x2="154.94" y2="104.14" width="0.1524" layer="91"/>
-</segment>
-</net>
+<pinref part="110INB" gate="G$1" pin="1"/>
+<wire x1="134.62" y1="116.84" x2="134.62" y2="104.14" width="0.1524" layer="91"/>
+<wire x1="134.62" y1="104.14" x2="147.32" y2="104.14" width="0.1524" layer="91"/>
+<junction x="147.32" y="104.14"/>
+</segment>
+</net>
