File: PCB/WaterCirculation/WaterCirculation.brd (EAGLE design)
At the start: 67 x 52.1 mm, 27 parts, among them K1 G5V1, K2 G5V1, K3 G5V1, Q1 MPSA42, Q3 MPSA42

Commit message: final layout
Parts:
- added 110INB: (no value), SparkFun-Connectors:SCREWTERMINAL-3.5MM-2
- moved LED2 17.3 mm to (45.7, 45.7)
- moved LED1 16.5 mm to (31.8, 45.7)
- moved R2 12.8 mm to (40.6, 61.0)
- moved R1 11.5 mm to (40.6, 66.0)
- moved D1 7.62 mm to (31.8, 66.0)
- moved D2 7.62 mm to (50.8, 66.0)
- moved Q1 7.62 mm to (31.8, 52.1)
- moved Q3 7.62 mm to (50.8, 52.1)
- moved R3 7.62 mm to (50.8, 57.1)
- moved R4 7.62 mm to (31.8, 57.1)
- moved R5 7.62 mm to (50.8, 62.2)
- moved R6 7.62 mm to (31.8, 62.2)
- moved K1 5.08 mm to (31.8, 74.9)
- moved K2 5.08 mm to (40.6, 74.9)
- moved K3 5.08 mm to (50.8, 74.9)
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Connections:
- net N$10: now also 110INB.1
- net N$6: now also 110INB.2
Other:
- board size 67 x 52.1 mm -> 65.7 x 54.6 mm
- board text added: "PWR IN"

Commit message: OSH Park Release
Routing:
- net +5V: track 0.00 -> 214.1 mm, vias 0 -> 2
- net GND: track 0.00 -> 172.8 mm
- net TEMP_DATA: track 0.00 -> 87.2 mm
- net N$5: track 0.00 -> 84.0 mm, vias 0 -> 1
- net N$3: track 0.00 -> 70.7 mm
- net N$7: track 0.00 -> 64.8 mm
- net +12V: track 0.00 -> 53.1 mm
- net N$4: track 0.00 -> 52.5 mm
- net PUMP: track 0.00 -> 52.2 mm
- net N$2: track 0.00 -> 40.8 mm, vias 0 -> 2
- net N$12: track 0.00 -> 38.4 mm
- net N$10: track 0.00 -> 30.8 mm
- net N$6: track 0.00 -> 26.1 mm
- net N$11: track 0.00 -> 20.6 mm
- net LED: track 0.00 -> 18.7 mm, vias 0 -> 1
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